File: uStar/uStar.sch (EAGLE design)
At the start: 45 parts, among them IC1 INA138, M1 Mount, M2 Mount, T1 NPN, 0.25A, U1 MAX4594EXK+T21-0076E-M, X1 MINI-USB-32005-201, X2 BU-SMA-V

Commit message: updated schematics and BOM with notes in the course of assembling the 3 main PCBs
Other:
- note added: "Radio Board"
- note removed: "umami"
- moved on the sheet: M1, M2
Changed lines of the file:
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@@
 Replace with trough hole when re-layout brd (11-29-2019)</text>
 <text x="142.24" y="132.08" size="1.778" layer="97">9DOF long pcb is obsolete,Garrett has old stock on hand</text>
+<text x="242.57" y="21.59" size="2.54" layer="97">Radio Board</text>
 </plain>
 <instances>
@@
 <attribute name="SHEET" x="240.665" y="1.27" size="2.54" layer="94"/>
 <attribute name="AUTHOR" x="229.87" y="11.43" size="2.54" layer="94"/>
-<attribute name="SHEET_NAME" x="172.72" y="1.27" size="2.54" layer="94"/>
-</instance>
-<instance part="M1" gate="G$1" x="189.14" y="32.18" smashed="yes">
-<attribute name="NAME" x="189.14" y="49.96" size="1.778" layer="95"/>
-<attribute name="VALUE" x="189.14" y="29.64" size="1.778" layer="96"/>
+</instance>
+<instance part="M1" gate="G$1" x="176.44" y="32.18" smashed="yes">
+<attribute name="NAME" x="176.44" y="49.96" size="1.778" layer="95"/>
+<attribute name="VALUE" x="176.44" y="29.64" size="1.778" layer="96"/>
 </instance>
 <instance part="D2" gate="G$1" x="205.34" y="69.74" smashed="yes" rot="R180">
@@
 </instance>
 <instance part="X1" gate="G$1" x="19.11" y="44.73" smashed="yes" rot="R180">
-<attribute name="NAME" x="19.11" y="33.3" size="1.778" layer="95" rot="R180"/>
+<attribute name="NAME" x="29.27" y="35.84" size="1.778" layer="95" rot="R180"/>
 <attribute name="VALUE" x="8.95" y="52.35" size="1.778" layer="96" rot="R270"/>
 <attribute name="NOTLOADED" x="19.11" y="44.73" size="1.778" layer="96" rot="R180" display="off"/>
@@
 <attribute name="VALUE" x="133.6" y="70.78" size="1.778" layer="96" rot="R180"/>
 </instance>
-<instance part="M2" gate="G$1" x="235.14" y="32.18" smashed="yes">
-<attribute name="NAME" x="235.14" y="49.96" size="1.778" layer="95"/>
-<attribute name="VALUE" x="235.14" y="29.64" size="1.778" layer="96"/>
+<instance part="M2" gate="G$1" x="222.44" y="32.18" smashed="yes">
+<attribute name="NAME" x="222.44" y="49.96" size="1.778" layer="95"/>
+<attribute name="VALUE" x="222.44" y="29.64" size="1.778" layer="96"/>
 </instance>
 <instance part="T1" gate="G$1" x="252" y="124.5" smashed="yes">
@@
 </instance>
 <instance part="R12" gate="G$1" x="149" y="164" smashed="yes" rot="R90">
-<attribute name="NAME" x="147.5014" y="160.19" size="1.778" layer="95" rot="R90"/>
+<attribute name="NAME" x="142.4214" y="160.19" size="1.778" layer="95" rot="R90"/>
 <attribute name="VALUE" x="152.302" y="160.19" size="1.778" layer="96" rot="R90"/>
 <attribute name="NOTLOADED" x="149" y="164" size="1.778" layer="96" rot="R90" display="off"/>
 </instance>
 <instance part="R10" gate="G$1" x="254.5" y="109" smashed="yes" rot="R90">
-<attribute name="NAME" x="253.0014" y="105.19" size="1.778" layer="95" rot="R90"/>
+<attribute name="NAME" x="247.9214" y="107.73" size="1.778" layer="95" rot="R90"/>
 <attribute name="VALUE" x="257.802" y="105.19" size="1.778" layer="96" rot="R90"/>
 <attribute name="NOTLOADED" x="254.5" y="109" size="1.778" layer="96" rot="R90" display="off"/>
@@
 </segment>
 <segment>
-<wire x1="209.46" y1="34.72" x2="212" y2="34.72" width="0.1524" layer="91"/>
+<wire x1="196.76" y1="34.72" x2="199.3" y2="34.72" width="0.1524" layer="91"/>
 <pinref part="M1" gate="G$1" pin="GND"/>
-<label x="212" y="34.72" size="1.27" layer="95" xref="yes"/>
+<label x="199.3" y="34.72" size="1.27" layer="95" xref="yes"/>
 </segment>
 <segment>
@@
 </segment>
 <segment>
-<wire x1="255.46" y1="34.72" x2="258" y2="34.72" width="0.1524" layer="91"/>
+<wire x1="242.76" y1="34.72" x2="245.3" y2="34.72" width="0.1524" layer="91"/>
 <pinref part="M2" gate="G$1" pin="GND"/>
-<label x="258" y="34.72" size="1.27" layer="95" xref="yes"/>
+<label x="245.3" y="34.72" size="1.27" layer="95" xref="yes"/>
 </segment>
 <segment>
@@
 </segment>
 <segment>
-<wire x1="209.46" y1="44.88" x2="212" y2="44.88" width="0.1524" layer="91"/>
+<wire x1="196.76" y1="44.88" x2="199.3" y2="44.88" width="0.1524" layer="91"/>
 <pinref part="M1" gate="G$1" pin="1WIRE"/>
-<label x="212" y="44.88" size="1.27" layer="95" xref="yes"/>
+<label x="199.3" y="44.88" size="1.27" layer="95" xref="yes"/>
 </segment>
 <segment>
@@
 </segment>
 <segment>
-<wire x1="255.46" y1="44.88" x2="258" y2="44.88" width="0.1524" layer="91"/>
+<wire x1="242.76" y1="44.88" x2="245.3" y2="44.88" width="0.1524" layer="91"/>
 <pinref part="M2" gate="G$1" pin="1WIRE"/>
-<label x="258" y="44.88" size="1.27" layer="95" xref="yes"/>
+<label x="245.3" y="44.88" size="1.27" layer="95" xref="yes"/>
 </segment>
 </net>
@@
 </segment>
 <segment>
-<wire x1="209.46" y1="42.34" x2="212" y2="42.34" width="0.1524" layer="91"/>
+<wire x1="196.76" y1="42.34" x2="199.3" y2="42.34" width="0.1524" layer="91"/>
 <pinref part="M1" gate="G$1" pin="VCC"/>
-<label x="212" y="42.34" size="1.27" layer="95" xref="yes"/>
-</segment>
-<segment>
-<wire x1="255.46" y1="42.34" x2="258" y2="42.34" width="0.1524" layer="91"/>
+<label x="199.3" y="42.34" size="1.27" layer="95" xref="yes"/>
+</segment>
+<segment>
+<wire x1="242.76" y1="42.34" x2="245.3" y2="42.34" width="0.1524" layer="91"/>
 <pinref part="M2" gate="G$1" pin="VCC"/>
-<label x="258" y="42.34" size="1.27" layer="95" xref="yes"/>
+<label x="245.3" y="42.34" size="1.27" layer="95" xref="yes"/>
 </segment>
 </net>
@@
 </segment>
 <segment>
-<wire x1="209.46" y1="39.8" x2="212" y2="39.8" width="0.1524" layer="91"/>
+<wire x1="196.76" y1="39.8" x2="199.3" y2="39.8" width="0.1524" layer="91"/>
 <pinref part="M1" gate="G$1" pin="EXT_VCC"/>
-<label x="212" y="39.8" size="1.27" layer="95" xref="yes"/>
+<label x="199.3" y="39.8" size="1.27" layer="95" xref="yes"/>
 </segment>
 </net>
@@
 </segment>
 <segment>
-<wire x1="255.46" y1="37.26" x2="258" y2="37.26" width="0.1524" layer="91"/>
-<label x="258" y="37.26" size="1.27" layer="95" xref="yes"/>
+<wire x1="242.76" y1="37.26" x2="245.3" y2="37.26" width="0.1524" layer="91"/>
+<label x="245.3" y="37.26" size="1.27" layer="95" xref="yes"/>
 <pinref part="M2" gate="G$1" pin="BATT_LEVEL"/>
 </segment>
@@
 <plain>
 <text x="116.84" y="154.94" size="6.4516" layer="97">RADIO</text>
-<text x="228.6" y="10.16" size="6.4516" layer="249">umami</text>
 <text x="147.32" y="142.24" size="1.778" layer="97">Digikey A97593-ND is similar to what's on sample board </text>
 <text x="147.32" y="144.78" size="1.778" layer="97">SMA : cant find prior order with thius part on it</text>
