File: BatteryV0.9/BattMonTimer.brd (EAGLE design)
At the start: 88 x 88 mm, 62 parts, among them IC1 TMP36GT9Z, IC2 TLV2211, IC3 INA138, IC4 TMP36GRT, IC6 CD74HC4060, IC7 74LVC1G74DCT, IC8 ICM7555SO08, M1 Mount, M2 Mount, P2 SSM3J338RSOT-23F_TOS-M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

Commit message: Added the cost of parts and Labor in the BOM
Routing:
- net UVP_TRIG: track 49.4 -> 54.5 mm
